File: pcb/pcb.kicad_pcb (KiCad board)
At the start: 2 copper layers, 137.5 x 93.4 mm, 52 parts, among them SW1 SW_SPST, SW10 SW_SPST, SW11 SW_SPST, SW12 SW_SPST, SW13 SW_SPST, SW14 SW_SPST, SW15 SW_SPST, SW16 SW_SPST, SW17 SW_SPST, SW18 SW_SPST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

Commit message: A v1.3
Other:
- board text added: "Ergonaut One A v1.3 by yumagulovrn"
- board text removed: "Ergonaut One v1.3 by yumagulovrn"

Commit message: final
move 2 ergo
Other:
- board text added: "Ergonaut One v1.3 by yumagulovrn"
- board text removed: "Ergonaut One A v1.3 by yumagulovrn"
